File: SwitchPi-v0.2.brd (EAGLE design)
At the start: 36.5 x 54.6 mm, 10 parts, among them IC1 MCP23017SP, IC2 MCP2300X/P, P2 P2, P3 P3

Commit message: updates
Parts:
- added RN1: 10K, resistor-net:RN-5
- P4: device adafruit:1X18 -> adafruit:1X18-BIG
- moved R4 10.2 mm to (24.1, 43.2)
- moved P2 2.54 mm to (35.6, 11.4)
- moved P3 2.54 mm to (35.6, 31.8)
Connections:
- net +5V: now also RN1.1
- net N$10: now also RN1.2
- net N$7: now also RN1.5
- net N$8: now also RN1.4
- net N$9: now also RN1.3
Routing:
- net GND: track 163.0 -> 0.00 mm
- net SDA: track 114.9 -> 62.0 mm
- net GPB7: track 42.7 -> 10.8 mm
- net GPB6: track 40.2 -> 10.5 mm, vias 2 -> 0
- net +5V: track 114.1 -> 120.8 mm
- net GPA2: track 30.0 -> 23.5 mm
- net SCL: track 53.4 -> 59.9 mm, vias 1 -> 0
- net GPA0: track 28.2 -> 23.5 mm, vias 1 -> 0
- net GPA4: track 20.9 -> 23.5 mm
- net N$9: track 6.35 -> 8.89 mm
- net N$8: track 6.35 -> 8.89 mm
- net N$7: track 6.35 -> 8.89 mm
- net N$6: track 6.35 -> 8.89 mm
- net N$4: track 6.35 -> 8.89 mm
- net N$2: track 6.35 -> 8.89 mm
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Other:
- board size 36.5 x 54.6 mm -> 39 x 54.6 mm
- board text removed: "(C)2013 Ken Rice <krice@freeswitch.org> This work is licensed under the Creative Commons Attribution-NonCommercial-ShareAlike 3.0 Unported License. To view a copy of this license, visit http://creativecommons.org/licenses/by-nc-sa/3.0/."
